File: PCB/RP2040 Devboard.kicad_pcb (KiCad board)
At the start: 2 copper layers, 32 x 52 mm, 32 parts, among them J1 USB_C_Receptacle_USB2.0_16P, J2 Conn_01x20, J3 Conn_01x20, J4 Conn_01x03, SW1 SW_Push, U1 RP2040, U2 MCP1700x-330xxTT, U4 W25Q16JVUXIQ TR, Y1 12 MHz

Commit message: Add files via upload
Parts:
- added D1: LED, LED_SMD:LED_0201_0603Metric, F.Cu at (158.9, 114.5)
- added D4: LED, LED_SMD:LED_0201_0603Metric, F.Cu at (159.0, 111.1)
- added D5: LED, LED_SMD:LED_0201_0603Metric, F.Cu at (159.1, 112.9)
- added J6: Conn_01x02_Pin, Connector_Hirose:Hirose_DF13-02P-1.25DSA_1x02_P1.25mm_Vertical, F.Cu at (151.5, 124.6)
- added R10: 1K, Resistor_SMD:R_0603_1608Metric, F.Cu at (161.5, 114.5)
- added R12: 1K, Resistor_SMD:R_0603_1608Metric, F.Cu at (161.8, 111.1)
- added R13: 1K, Resistor_SMD:R_0603_1608Metric, F.Cu at (161.8, 112.9)
- R1, R2, R3, R4: footprint Resistor_SMD:R_0201_0603Metric_Pad0.64x0.40mm_HandSolder -> Capacitor_SMD:C_0603_1608Metric
- moved R3 0.31 mm to (158.9, 118.6)
- moved R4 0.11 mm to (163.3, 118.7)
Routing:
- net GPIO22: track 15.6 -> 32.4 mm, vias 2 -> 3
- net GPIO10: track 18.6 -> 34.5 mm, vias 0 -> 1
- net Power: track 19.1 -> 28.0 mm
- net 3.3V: track 105.2 -> 108.5 mm
- net Net-(D5-A): track 0.00 -> 1.61 mm
- net GND: track 155.0 -> 153.6 mm
- net Net-(D1-A): track 0.00 -> 1.42 mm
- net GPIO11: track 21.6 -> 20.7 mm
