File: PCB/RP2040 Devboard.kicad_sch (KiCad schematic)
At the start: 32 parts, among them J1 USB_C_Receptacle_USB2.0_16P, J2 Conn_01x20, J3 Conn_01x20, J4 Conn_01x03, SW1 SW_Push, U1 RP2040, U2 MCP1700x-330xxTT, U4 W25Q16JVUXIQ TR, Y1 12 MHz

Commit message: Add files via upload
Parts:
- added D1, D4, D5: LED, LED_SMD:LED_0201_0603Metric, symbol Device:LED
- added J6: Conn_01x02_Pin, Connector_Hirose:Hirose_DF13-02P-1.25DSA_1x02_P1.25mm_Vertical, symbol Connector:Conn_01x02_Pin
- added R10, R12, R13: 1K, Resistor_SMD:R_0603_1608Metric, symbol Device:R
- R1, R2, R3, R4: footprint Resistor_SMD:R_0201_0603Metric_Pad0.64x0.40mm_HandSolder -> Capacitor_SMD:C_0603_1608Metric
Connections:
- net 3.3V: now also R10.1
- net GND: now also D1.1 (K), D4.1 (K), D5.1 (K), J6.1 (Pin_1)
- net GPIO10: now also R12.1
- net GPIO22: now also R13.1
- net Power: now also J6.2 (Pin_2)
- new net: D5.2 (A), R13.2
- new net: D1.2 (A), R10.2
- new net: D4.2 (A), R12.2
